File: pcb/destilador_pcb.brd (EAGLE design)
At the start: 160 x 100 mm, 26 parts, among them Q1 IRF540, Q2 IRF540, T2 BTA26-V

Commit message: PCB finalizada
Parts:
- removed D1, D2: 1N4004, diode:DO41-10
- moved R1 25.2 mm to (-59.7, 26.7), turned to 90 degrees
- moved OK1 21.8 mm to (-41.9, 38.1), turned to 0 degrees
- moved R5 19.8 mm to (-55.9, 26.7), turned to 90 degrees
- moved B2 14.0 mm to (-41.9, 19.1)
- moved R4 11.7 mm to (-53.3, 19.1)
- moved R8 11.4 mm to (-78.7, 27.9)
- moved R7 7.73 mm to (-73.7, 27.9)
- moved Q2 5.08 mm to (-68.6, 39.4)
- moved R2 4.02 mm to (-54.6, 43.2)
- moved R3 4.02 mm to (-59.7, 43.2)
- moved T2 1.27 mm to (-36.8, 6.35)
- moved AC_IN 1.27 mm to (-30.5, 35.6)
- moved X2 1.27 mm to (-30.5, 25.4)
- moved LED1 1.27 mm to (-66.0, 20.3)
Connections:
- removed net PIN_4: PCB1.4, Q2.G, R7.1
- removed net PIN_5: PCB1.5, Q1.G, R8.2
- new net PIN_8: PCB1.8, Q2.G, R7.1
- new net PIN_9: PCB1.9, Q1.G, R8.2
- net GND: no longer D1.A, D2.A
- net N$11: no longer D1.C
- net N$15: no longer D2.C
Routing:
- net GND: track 25.2 -> 115.5 mm, vias 0 -> 4
- net 5V: track 62.6 -> 102.9 mm
- net PIN_4: track 33.9 -> 0.00 mm
- net PIN_9: track 0.00 -> 25.9 mm
- net PIN_8: track 0.00 -> 25.0 mm
- net PIN_2: track 7.93 -> 23.2 mm
- net N$2: track 27.5 -> 39.0 mm
- net N$5: track 31.8 -> 20.6 mm
- net N$3: track 24.7 -> 13.8 mm
- net N$11: track 17.9 -> 8.66 mm
- net N$8: track 11.2 -> 5.61 mm
- net N$4: track 17.3 -> 23.0 mm
- net N$6: track 26.0 -> 20.4 mm
- net PIN_5: track 5.39 -> 0.00 mm
- net N$1: track 38.6 -> 42.2 mm
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Other:
- board size 160 x 100 mm -> 101.6 x 53.3 mm
