File: pcb/destilador_pcb.sch (EAGLE design)
At the start: 26 parts, among them Q1 IRF540, Q2 IRF540, T2 BTA26-V

Commit message: PCB finalizada
Parts:
- removed D1, D2: 1N4004, diode:1N4004
Connections:
- removed net PIN_4: PCB1.4, Q2.G, R7.1
- removed net PIN_5: PCB1.5, Q1.G, R8.2
- new net PIN_8: PCB1.8, Q2.G, R7.1
- new net PIN_9: PCB1.9, Q1.G, R8.2
- net GND: no longer D1.A, D2.A
- net N$11: no longer D1.C
- net N$15: no longer D2.C
